File: kicad/g100s.kicad_pcb (KiCad board)
At the start: 2 copper layers, 77.4 x 46 mm, 38 parts, among them J1 Conn_01x05_Female, J2 Conn_01x02_Female, J3 Conn_01x03_Female, SW1 SW_SPDT, SW2 SW_SPDT, SW3 SW_SPDT, SW4 SW_SPDT, SW5 SW_SPDT, SW6 SW_SPDT, SW7 SW_SPST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

Commit message: update kicad files
Parts:
- C9: value 4.7uF -> 100nF
Changed lines of the file:
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@@
       (effects (font (size 1 1) (thickness 0.15)))
     )
-    (fp_text value "4.7uF" (at 0 1.68 -270) (layer "F.Fab")
+    (fp_text value "100nF" (at 0 1.68 -270) (layer "F.Fab")
       (effects (font (size 1 1) (thickness 0.15)))
     )

Commit message: update kicad files
Parts:
- moved C7 1.37 mm to (104.8, 145.2), turned to -90 degrees
- moved C1 1.16 mm to (87.5, 138.2)
- moved C8 0.87 mm to (88.1, 141.3)
- moved C13 0.23 mm to (80.0, 137.9)
- moved R1 0.08 mm to (84.6, 135.5)
- moved R2 0.08 mm to (84.6, 133.5)
- moved C12 0.06 mm to (80.0, 135.6)
Routing:
- net GND: track 178.9 -> 129.2 mm, vias 14 -> 15
- net VCC: track 169.5 -> 167.8 mm
- net Net-(C1-Pad2): track 3.07 -> 4.27 mm
- net VDD: track 70.6 -> 71.1 mm
- net MOSI-H: track 36.1 -> 35.6 mm

Commit message: remove sidebuttons
Parts:
- removed the SW4 at (86.8, 162.9)
- removed SW5: SW_SPDT, mouse:Microswitch_SPDT_D2F
- renumbered SW6 to SW4
Connections:
- U1 pad 21: +rsb -> +dpi
- U1 pad 22: +dpi -> no_connect_(U1-Pad22)
- U1 pad 25: +fsb -> no_connect_(U1-Pad25)
- U1 pad 36: -dpi -> no_connect_(U1-Pad36)
- U1 pad 37: -fsb -> no_connect_(U1-Pad37)
- U1 pad 38: -rsb -> -dpi
Routing:
- net -fsb: track 78.7 -> 0.00 mm
- net GND: track 129.2 -> 54.4 mm, vias 15 -> 14
- net +fsb: track 67.3 -> 0.00 mm, vias 1 -> 0
- net -rsb: track 62.3 -> 0.00 mm
- net +rsb: track 43.3 -> 0.00 mm, vias 1 -> 0
- net -middle: track 104.7 -> 102.2 mm
- net WHL_LED: track 95.8 -> 94.1 mm
- net -dpi: track 52.3 -> 50.9 mm
- net +dpi: track 91.1 -> 89.8 mm
